Commit message: modified:   .vscode/c_cpp_properties.json 	modified:   .vscode/settings.json 	modified:   omni_control/include/omni_control/reach_goal.hpp 	modified:   omni_control/src/reach_goal.cpp 	modified:   omni_control/src/reach_goal_node.cpp 	modified:   omni_description/config/omnidirectional_controller.yaml 	modified:   omni_description/urdf/omni.urdf.xacro 	modified:   omni_description/urdf/omni_base.xacro 	modified:   omni_description/urdf/omni_base_gazebo.xacro

File: omni_description/urdf/omni.urdf.xacro (robot description, xacro)
@@ -2,10 +2,6 @@
 <robot name="omni" xmlns:xacro="http://www.ros.org/wiki/xacro">
     <xacro:include filename="common_properties.xacro" />
-<<<<<<< HEAD
     <!-- <xacro:include filename="omni_base.xacro" /> -->
     <xacro:include filename="omni_base_wheels.xacro" />
-=======
-    <xacro:include filename="omni_base.xacro" />
->>>>>>> origin/TUF
     <xacro:include filename="omni_base_gazebo.xacro" />
 </robot>

File: omni_description/urdf/omni_base.xacro (robot description, xacro)
@@ -4,9 +4,5 @@
     <xacro:property name="base_length" value="0.15" />
     <xacro:property name="wheel_radius" value="0.05" />
-<<<<<<< HEAD
     <xacro:property name="wheel_length" value="0.036" />
-=======
-    <xacro:property name="wheel_length" value="0.04" />
->>>>>>> origin/TUF
     <link name="base_footprint" />
     <link name="base_link">
@@ -24,9 +20,5 @@
             <origin xyz="0 0 ${base_length / 2.0}" rpy="0 0 0" />
         </collision>
-<<<<<<< HEAD
         <xacro:cylinder_inertia m="2.0" r="${base_radius}" l ="${base_length}"
-=======
-        <xacro:cylinder_inertia m="5.0" r="${base_radius}" l ="${base_length}"
->>>>>>> origin/TUF
                            xyz="0 0 0" rpy="0 0 0" />
     </link>

File: omni_description/urdf/omni_base_gazebo.xacro (robot description, xacro)
@@ -20,10 +20,6 @@
     </gazebo>
     <xacro:macro name="ros2_control_wheel_joint" params="suffix">
-<<<<<<< HEAD
         <!-- <joint name="base_wheel_${suffix}_joint"> -->
         <joint name="wheel${suffix}_joint">
-=======
-        <joint name="base_wheel_${suffix}_joint">
->>>>>>> origin/TUF
             <command_interface name="velocity">
                 <param name="initial_value">0</param>
